Commit message: fix(gripper): increase friction coefficients to prevent object slipping

File: ws_thor/src/thor_urdf/urdf/thor_gazebo.xacro (robot description, xacro)
@@ -8,3 +8,34 @@
         </plugin>
     </gazebo>
+    <!-- ===== Gripper Finger Friction & Contact Properties ===== -->
+    <!-- Right Finger -->
+    <gazebo reference="gripper_finger_right">
+        <mu1>1.5</mu1>
+        <mu2>1.5</mu2>
+        <kp>1000000.0</kp>
+        <kd>100.0</kd>
+        <minDepth>0.001</minDepth>
+        <maxVel>0.01</maxVel>
+        <selfCollide>false</selfCollide>
+        <material>Gazebo/DarkGrey</material>
+    </gazebo>
+    <!-- Left Finger -->
+    <gazebo reference="gripper_finger_left">
+        <mu1>1.5</mu1>
+        <mu2>1.5</mu2>
+        <kp>1000000.0</kp>
+        <kd>100.0</kd>
+        <minDepth>0.001</minDepth>
+        <maxVel>0.01</maxVel>
+        <selfCollide>false</selfCollide>
+        <material>Gazebo/DarkGrey</material>
+    </gazebo>
+    <!-- Gripper base (link_5) also benefits from contact tuning -->
+    <gazebo reference="link_5">
+        <mu1>1.0</mu1>
+        <mu2>1.0</mu2>
+        <kp>1000000.0</kp>
+        <kd>100.0</kd>
+        <minDepth>0.001</minDepth>
+    </gazebo>
 </robot>
