Commit message: refactor: update IKControls configuration and clean up stale build artifacts

File: ws_thor/install/thor_urdf/share/thor_urdf/urdf/thor.urdf.xacro (robot description, xacro)
@@ -241,5 +241,5 @@
         <origin xyz="0.009742 0.081458 0.0" rpy="0 0 0"/>
         <axis xyz="-0.0 0.0 1.0"/>
-        <limit lower="-0.5" upper="0.5" effort="10.0" velocity="2.0"/>
+        <limit lower="-0.75" upper="0.5" effort="1.5" velocity="2.0"/>
     </joint>
     <joint name="gripperbase_to_armgearleft" type="revolute">
@@ -248,5 +248,5 @@
         <origin xyz="-0.009743 0.081458 0.0" rpy="0 0 0"/>
         <axis xyz="-0.0 0.0 1.0"/>
-        <limit lower="-0.5" upper="0.5" effort="10.0" velocity="2.0"/>
+        <limit lower="-0.75" upper="0.5" effort="1.5" velocity="2.0"/>
         <mimic joint="gripperbase_to_armgearright" multiplier="-1"/>
     </joint>

File: ws_thor/install/thor_urdf/share/thor_urdf/urdf/thor_gazebo.xacro (robot description, xacro)
@@ -11,10 +11,10 @@
     <!-- Right Finger -->
     <gazebo reference="gripper_finger_right">
-        <mu1>100</mu1>
-        <mu2>100</mu2>
+        <mu1>100.0</mu1>
+        <mu2>100.0</mu2>
         <kp>1000000.0</kp>
         <kd>100.0</kd>
-        <minDepth>0.001</minDepth>
-        <maxVel>0.01</maxVel>
+        <minDepth>0.002</minDepth>
+        <maxVel>0.0</maxVel>
         <selfCollide>false</selfCollide>
         <material>Gazebo/DarkGrey</material>
@@ -22,10 +22,10 @@
     <!-- Left Finger -->
     <gazebo reference="gripper_finger_left">
-        <mu1>100</mu1>
-        <mu2>100</mu2>
+        <mu1>100.0</mu1>
+        <mu2>100.0</mu2>
         <kp>1000000.0</kp>
         <kd>100.0</kd>
-        <minDepth>0.001</minDepth>
-        <maxVel>0.01</maxVel>
+        <minDepth>0.002</minDepth>
+        <maxVel>0.0</maxVel>
         <selfCollide>false</selfCollide>
         <material>Gazebo/DarkGrey</material>
