Commit message: refactor: update robot joint limits

File: ws_gryphon/src/gryphon_moveit/config/gryphon_arm.urdf (robot description, URDF)
Before this commit: robot gryphon_arm, 10 links, 9 joints
Joints:
- joint gripperbase_to_armgearleft: limit lower=-0.5 upper=0.5 effort=10.0 velocity=2.0 -> lower=-0.7 upper=0.7 effort=10.0 velocity=2.0
- joint gripperbase_to_armgearright: limit lower=-0.5 upper=0.5 effort=10.0 velocity=2.0 -> lower=-0.7 upper=0.7 effort=10.0 velocity=2.0
