Commit message: refactor: migrate simulation stack from Gazebo Classic to Ignition Gazebo (gz_sim)

File: ws_gryphon/src/gryphon_urdf/urdf/gryphon_arm.ros2_control.xacro (robot description, xacro)
@@ -5,5 +5,5 @@
     <xacro:if value="$(arg is_sim)">
         <hardware>
-            <plugin>gazebo_ros2_control/GazeboSystem</plugin>
+            <plugin>ign_ros2_control/IgnitionSystem</plugin>
         </hardware>
         <joint name="gripperbase_to_armgearleft">

File: ws_gryphon/src/gryphon_urdf/urdf/gryphon_gazebo.xacro (robot description, xacro)
@@ -1,6 +1,7 @@
 <?xml version="1.0"?>
 <robot xmlns:xacro="http://www.ros.org/wiki/xacro" name="gryphon_arm">
+    <!-- Ignition Gazebo: gz_ros2_control plugin -->
     <gazebo>
-        <plugin filename="libgazebo_ros2_control.so" name="gazebo_ros2_control">
+        <plugin filename="libign_ros2_control-system.so" name="ign_ros2_control::IgnitionROS2ControlPlugin">
             <robot_param>robot_description</robot_param>
             <robot_param_node>robot_state_publisher</robot_param_node>
@@ -18,5 +19,4 @@
         <maxVel>0.0</maxVel>
         <selfCollide>false</selfCollide>
-        <material>Gazebo/DarkGrey</material>
     </gazebo>
     <!-- Left Finger -->
@@ -29,5 +29,4 @@
         <maxVel>0.0</maxVel>
         <selfCollide>false</selfCollide>
-        <material>Gazebo/DarkGrey</material>
     </gazebo>
     <!-- Gripper base (link_5) also benefits from contact tuning -->
